File: teensy_to_em3242.kicad_pcb (KiCad board)
At the start: 2 copper layers, 43.2 x 50.8 mm, 9 parts, among them J1 PIN_ARRAY_3X1, J2 PIN_ARRAY_3X1, J3 PIN_ARRAY_3X1, J4 PIN_ARRAY_3X1, M1 VAL**, M2 VAL**, M3 VAL**, M4 VAL**, U1 TEENSY3.1

Commit message: Shortened board so that it is less the 50mm x 50mm. Added markings for pin #1 on sensor headers.
Parts:
- moved M3 1.27 mm to (90.8, 97.2)
- moved M4 1.27 mm to (54.0, 97.2)
Other:
- board size 43.2 x 50.8 mm -> 43.2 x 49.5 mm
Changed lines of the file:
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@@
     (area 50.724999 50.724999 94.055001 101.675001)
     (thickness 1.6)
-    (drawings 13)
+    (drawings 27)
     (tracks 48)
     (zones 0)
@@
   )
   (module hole_4-40:MOUNT_HOLE_4_40 (layer F.Cu)
-    (at 90.805 98.425)
+    (at 90.805 97.155)
     (fp_text reference M3 (at 0 -2.032) (layer F.SilkS) hide
       (effects (font (size 0.254 0.254) (thickness 0.0635)))
@@
   )
   (module hole_4-40:MOUNT_HOLE_4_40 (layer F.Cu)
-    (at 53.975 98.425)
+    (at 53.975 97.155)
     (fp_text reference M4 (at 0 -2.032) (layer F.SilkS) hide
       (effects (font (size 0.254 0.254) (thickness 0.0635)))
@@
     (pad "" thru_hole circle (at 0 0) (size 3.302 3.302) (drill 3.048) (layers *.Cu *.SilkS *.Mask))
   )
+  (dimension 49.53 (width 0.3) (layer Dwgs.User)
+    (gr_text "49.530 mm" (at 101.68 75.565 270) (layer Dwgs.User)
+      (effects (font (size 1.5 1.5) (thickness 0.3)))
+    )
+    (feature1 (pts (xy 90.805 100.33) (xy 103.03 100.33)))
+    (feature2 (pts (xy 90.805 50.8) (xy 103.03 50.8)))
+    (crossbar (pts (xy 100.33 50.8) (xy 100.33 100.33)))
+    (arrow1a (pts (xy 100.33 100.33) (xy 99.743579 99.203496)))
+    (arrow1b (pts (xy 100.33 100.33) (xy 100.916421 99.203496)))
+    (arrow2a (pts (xy 100.33 50.8) (xy 99.743579 51.926504)))
+    (arrow2b (pts (xy 100.33 50.8) (xy 100.916421 51.926504)))
+  )
+  (dimension 43.18 (width 0.3) (layer Dwgs.User)
+    (gr_text "43.180 mm" (at 72.39 42.465) (layer Dwgs.User)
+      (effects (font (size 1.5 1.5) (thickness 0.3)))
+    )
+    (feature1 (pts (xy 93.98 53.975) (xy 93.98 41.115)))
+    (feature2 (pts (xy 50.8 53.975) (xy 50.8 41.115)))
+    (crossbar (pts (xy 50.8 43.815) (xy 93.98 43.815)))
+    (arrow1a (pts (xy 93.98 43.815) (xy 92.853496 44.401421)))
+    (arrow1b (pts (xy 93.98 43.815) (xy 92.853496 43.228579)))
+    (arrow2a (pts (xy 50.8 43.815) (xy 51.926504 44.401421)))
+    (arrow2b (pts (xy 50.8 43.815) (xy 51.926504 43.228579)))
+  )
+  (gr_line (start 93.98 53.975) (end 93.98 97.155) (angle 90) (layer Edge.Cuts) (width 0.15))
+  (gr_line (start 50.8 53.975) (end 50.8 97.155) (angle 90) (layer Edge.Cuts) (width 0.15))
+  (gr_line (start 87.376 64.516) (end 87.376 66.04) (angle 90) (layer F.SilkS) (width 0.2))
+  (gr_line (start 88.138 65.278) (end 87.376 64.516) (angle 90) (layer F.SilkS) (width 0.2))
+  (gr_line (start 88.138 65.278) (end 87.376 66.04) (angle 90) (layer F.SilkS) (width 0.2))
+  (gr_line (start 87.376 73.406) (end 87.376 74.93) (angle 90) (layer F.SilkS) (width 0.2))
+  (gr_line (start 88.138 74.168) (end 87.376 73.406) (angle 90) (layer F.SilkS) (width 0.2))
+  (gr_line (start 88.138 74.168) (end 87.376 74.93) (angle 90) (layer F.SilkS) (width 0.2))
+  (gr_line (start 87.376 82.296) (end 87.376 83.82) (angle 90) (layer F.SilkS) (width 0.2))
+  (gr_line (start 88.138 83.058) (end 87.376 82.296) (angle 90) (layer F.SilkS) (width 0.2))
+  (gr_line (start 88.138 83.058) (end 87.376 83.82) (angle 90) (layer F.SilkS) (width 0.2))
+  (gr_line (start 87.376 91.186) (end 87.376 92.71) (angle 90) (layer F.SilkS) (width 0.2))
+  (gr_line (start 88.138 91.948) (end 87.376 91.186) (angle 90) (layer F.SilkS) (width 0.2))
+  (gr_line (start 88.138 91.948) (end 87.376 92.71) (angle 90) (layer F.SilkS) (width 0.2))
   (gr_text A2 (at 86.995 71.12 90) (layer F.SilkS)
     (effects (font (size 1.5 1.5) (thickness 0.3)))
@@
     (effects (font (size 1.5 1.5) (thickness 0.3)))
   )
-  (gr_line (start 90.805 101.6) (end 53.975 101.6) (angle 90) (layer Edge.Cuts) (width 0.15))
+  (gr_line (start 90.805 100.33) (end 53.975 100.33) (angle 90) (layer Edge.Cuts) (width 0.15))
   (gr_line (start 53.975 50.8) (end 90.805 50.8) (angle 90) (layer Edge.Cuts) (width 0.15))
-  (gr_line (start 93.98 98.425) (end 93.98 53.975) (angle 90) (layer Edge.Cuts) (width 0.15))
-  (gr_line (start 50.8 53.975) (end 50.8 98.425) (angle 90) (layer Edge.Cuts) (width 0.15))
-  (gr_arc (start 53.975 98.425) (end 53.975 101.6) (angle 90) (layer Edge.Cuts) (width 0.15))
-  (gr_arc (start 90.805 98.425) (end 93.98 98.425) (angle 90) (layer Edge.Cuts) (width 0.15))
+  (gr_arc (start 53.975 97.155) (end 53.975 100.33) (angle 90) (layer Edge.Cuts) (width 0.15))
+  (gr_arc (start 90.805 97.155) (end 93.98 97.155) (angle 90) (layer Edge.Cuts) (width 0.15))
   (gr_arc (start 90.805 53.975) (end 90.805 50.8) (angle 90) (layer Edge.Cuts) (width 0.15))
   (gr_arc (start 53.975 53.975) (end 50.8 53.975) (angle 90) (layer Edge.Cuts) (width 0.15))
